File: apple_peeler_pcb/power_supply.kicad_sch (KiCad schematic)
At the start: 14 parts, among them J7 Header_01x02, U4 TPS562242

Commit message: prepare for fab
Parts:
- L1: value 2.2μH -> 4.7μH; LCSC C279946 -> C43183; MPN SWPA5020S2R2MT -> SWPA5020S4R7MT
- R35: value 1.5kΩ -> 15kΩ; LCSC C4310 -> C17475; MPN R 1.5kΩ 125mW 0805 -> R 15kΩ 125mW 0805
- U4: value TPS562242 -> TPS563206; LCSC C19272253 -> C22427434; MPN TPS562242DRLR -> TPS563206DRLR
Changed lines of the file:
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@@
 			)
 		)
-		(property "Value" "1.5kΩ"
+		(property "Value" "15kΩ"
 			(at 152.4 87.6299 0)
 			(effects
@@
 			)
 		)
-		(property "LCSC" "C4310"
+		(property "LCSC" "C17475"
 			(at 154.94 86.36 0)
 			(effects
@@
 			)
 		)
-		(property "MPN" "R 1.5kΩ 125mW 0805"
+		(property "MPN" "R 15kΩ 125mW 0805"
 			(at 154.94 86.36 0)
 			(effects
@@
 			)
 		)
-		(property "Value" "TPS562242"
+		(property "Value" "TPS563206"
 			(at 121.92 74.93 0)
 			(effects
@@
 			)
 		)
-		(property "LCSC" "C19272253"
+		(property "LCSC" "C22427434"
 			(at 121.92 82.55 0)
 			(effects
@@
 			)
 		)
-		(property "MPN" "TPS562242DRLR"
+		(property "MPN" "TPS563206DRLR"
 			(at 121.92 82.55 0)
 			(effects
@@
 			)
 		)
-		(property "Value" "2.2μH"
+		(property "Value" "4.7μH"
 			(at 147.32 77.47 90)
 			(effects
@@
 			)
 		)
-		(property "LCSC" "C279946"
+		(property "LCSC" "C43183"
 			(at 147.32 80.01 90)
 			(effects
@@
 			)
 		)
-		(property "MPN" "SWPA5020S2R2MT"
+		(property "MPN" "SWPA5020S4R7MT"
 			(at 147.32 80.01 90)
 			(effects
