File: apple_peeler_pcb/cec_interface.kicad_sch (KiCad schematic)
At the start: 7 parts, among them Q11 2N7002

Commit message: replace fancy debug connectors by pin header to save $8
Parts:
- renumbered R31 to R32, R32 to R33, R33 to R34, R34 to R35
Changed lines of the file:
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@@
 		(dnp no)
 		(fields_autoplaced yes)
-		(property "Reference" "R33"
+		(property "Reference" "R34"
 			(at 132.08 85.0899 0)
 			(effects
@@
 			(project "apple_peeler_pcb"
 				(path "/d5946b96-44a8-4a28-8641-19803e1510af/ab4760da-4146-4688-a275-418314974b55/81932bd6-0e7a-4e3b-bdf1-28d2dccc0222"
-					(reference "R33")
-					(unit 1)
-				)
-				(path "/d5946b96-44a8-4a28-8641-19803e1510af/ab4760da-4146-4688-a275-418314974b55/9898d91a-fb1c-440b-9509-02fc004394d7"
-					(reference "R59")
+					(reference "R34")
+					(unit 1)
+				)
+				(path "/d5946b96-44a8-4a28-8641-19803e1510af/ab4760da-4146-4688-a275-418314974b55/9898d91a-fb1c-440b-9509-02fc004394d7"
+					(reference "R60")
 					(unit 1)
 				)
@@
 		(on_board yes)
 		(dnp no)
-		(property "Reference" "#PWR058"
+		(property "Reference" "#PWR057"
 			(at 154.94 109.22 0)
 			(effects
@@
 			(project "apple_peeler_pcb"
 				(path "/d5946b96-44a8-4a28-8641-19803e1510af/ab4760da-4146-4688-a275-418314974b55/81932bd6-0e7a-4e3b-bdf1-28d2dccc0222"
-					(reference "#PWR058")
-					(unit 1)
-				)
-				(path "/d5946b96-44a8-4a28-8641-19803e1510af/ab4760da-4146-4688-a275-418314974b55/9898d91a-fb1c-440b-9509-02fc004394d7"
-					(reference "#PWR0127")
+					(reference "#PWR057")
+					(unit 1)
+				)
+				(path "/d5946b96-44a8-4a28-8641-19803e1510af/ab4760da-4146-4688-a275-418314974b55/9898d91a-fb1c-440b-9509-02fc004394d7"
+					(reference "#PWR0125")
 					(unit 1)
 				)
@@
 		(on_board yes)
 		(dnp no)
-		(property "Reference" "#PWR056"
+		(property "Reference" "#PWR055"
 			(at 134.62 83.82 0)
 			(effects
@@
 			(project "apple_peeler_pcb"
 				(path "/d5946b96-44a8-4a28-8641-19803e1510af/ab4760da-4146-4688-a275-418314974b55/81932bd6-0e7a-4e3b-bdf1-28d2dccc0222"
-					(reference "#PWR056")
-					(unit 1)
-				)
-				(path "/d5946b96-44a8-4a28-8641-19803e1510af/ab4760da-4146-4688-a275-418314974b55/9898d91a-fb1c-440b-9509-02fc004394d7"
-					(reference "#PWR0125")
+					(reference "#PWR055")
+					(unit 1)
+				)
+				(path "/d5946b96-44a8-4a28-8641-19803e1510af/ab4760da-4146-4688-a275-418314974b55/9898d91a-fb1c-440b-9509-02fc004394d7"
+					(reference "#PWR0123")
 					(unit 1)
 				)
@@
 		(on_board yes)
 		(dnp no)
-		(property "Reference" "R31"
+		(property "Reference" "R32"
 			(at 115.57 105.41 90)
 			(effects
@@
 			(project "apple_peeler_pcb"
 				(path "/d5946b96-44a8-4a28-8641-19803e1510af/ab4760da-4146-4688-a275-418314974b55/81932bd6-0e7a-4e3b-bdf1-28d2dccc0222"
-					(reference "R31")
-					(unit 1)
-				)
-				(path "/d5946b96-44a8-4a28-8641-19803e1510af/ab4760da-4146-4688-a275-418314974b55/9898d91a-fb1c-440b-9509-02fc004394d7"
-					(reference "R57")
+					(reference "R32")
+					(unit 1)
+				)
+				(path "/d5946b96-44a8-4a28-8641-19803e1510af/ab4760da-4146-4688-a275-418314974b55/9898d91a-fb1c-440b-9509-02fc004394d7"
+					(reference "R58")
 					(unit 1)
 				)
@@
 		(on_board yes)
 		(dnp no)
-		(property "Reference" "#PWR055"
+		(property "Reference" "#PWR054"
 			(at 121.92 129.54 0)
 			(effects
@@
 			(project "apple_peeler_pcb"
 				(path "/d5946b96-44a8-4a28-8641-19803e1510af/ab4760da-4146-4688-a275-418314974b55/81932bd6-0e7a-4e3b-bdf1-28d2dccc0222"
-					(reference "#PWR055")
-					(unit 1)
-				)
-				(path "/d5946b96-44a8-4a28-8641-19803e1510af/ab4760da-4146-4688-a275-418314974b55/9898d91a-fb1c-440b-9509-02fc004394d7"
-					(reference "#PWR0124")
+					(reference "#PWR054")
+					(unit 1)
+				)
+				(path "/d5946b96-44a8-4a28-8641-19803e1510af/ab4760da-4146-4688-a275-418314974b55/9898d91a-fb1c-440b-9509-02fc004394d7"
+					(reference "#PWR0122")
 					(unit 1)
 				)
@@
 		(dnp no)
 		(fields_autoplaced yes)
-		(property "Reference" "R34"
+		(property "Reference" "R35"
 			(at 147.32 85.09 90)
 			(effects
@@
 			(project "apple_peeler_pcb"
 				(path "/d5946b96-44a8-4a28-8641-19803e1510af/ab4760da-4146-4688-a275-418314974b55/81932bd6-0e7a-4e3b-bdf1-28d2dccc0222"
-					(reference "R34")
-					(unit 1)
-				)
-				(path "/d5946b96-44a8-4a28-8641-19803e1510af/ab4760da-4146-4688-a275-418314974b55/9898d91a-fb1c-440b-9509-02fc004394d7"
-					(reference "R60")
+					(reference "R35")
+					(unit 1)
+				)
+				(path "/d5946b96-44a8-4a28-8641-19803e1510af/ab4760da-4146-4688-a275-418314974b55/9898d91a-fb1c-440b-9509-02fc004394d7"
+					(reference "R61")
 					(unit 1)
 				)
@@
 		(on_board yes)
 		(dnp no)
-		(property "Reference" "#PWR057"
+		(property "Reference" "#PWR056"
 			(at 134.62 129.54 0)
 			(effects
@@
 			(project "apple_peeler_pcb"
 				(path "/d5946b96-44a8-4a28-8641-19803e1510af/ab4760da-4146-4688-a275-418314974b55/81932bd6-0e7a-4e3b-bdf1-28d2dccc0222"
-					(reference "#PWR057")
-					(unit 1)
-				)
-				(path "/d5946b96-44a8-4a28-8641-19803e1510af/ab4760da-4146-4688-a275-418314974b55/9898d91a-fb1c-440b-9509-02fc004394d7"
-					(reference "#PWR0126")
+					(reference "#PWR056")
+					(unit 1)
+				)
+				(path "/d5946b96-44a8-4a28-8641-19803e1510af/ab4760da-4146-4688-a275-418314974b55/9898d91a-fb1c-440b-9509-02fc004394d7"
+					(reference "#PWR0124")
 					(unit 1)
 				)
@@
 		(on_board yes)
 		(dnp no)
-		(property "Reference" "R32"
+		(property "Reference" "R33"
 			(at 123.19 116.84 0)
 			(effects
@@
 			(project "apple_peeler_pcb"
 				(path "/d5946b96-44a8-4a28-8641-19803e1510af/ab4760da-4146-4688-a275-418314974b55/81932bd6-0e7a-4e3b-bdf1-28d2dccc0222"
-					(reference "R32")
-					(unit 1)
-				)
-				(path "/d5946b96-44a8-4a28-8641-19803e1510af/ab4760da-4146-4688-a275-418314974b55/9898d91a-fb1c-440b-9509-02fc004394d7"
-					(reference "R58")
-					(unit 1)
-				)
+					(reference "R33")
+					(unit 1)
+				)
+				(path "/d5946b96-44a8-4a28-8641-19803e1510af/ab4760da-4146-4688-a275-418314974b55/9898d91a-fb1c-440b-9509-02fc004394d7"
+					(reference "R59")
+					(unit 1)
+				)
