File: apple_peeler_pcb/line_sense.kicad_sch (KiCad schematic)
At the start: 4 parts, among them Q8 2N7002

Commit message: replace fancy debug connectors by pin header to save $8
Parts:
- renumbered R22 to R23, R23 to R24, R24 to R25
Changed lines of the file:
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@@
 		(on_board yes)
 		(dnp no)
-		(property "Reference" "#PWR046"
+		(property "Reference" "#PWR045"
 			(at 135.89 116.84 0)
 			(effects
@@
 			(project "apple_peeler_pcb"
 				(path "/d5946b96-44a8-4a28-8641-19803e1510af/ab4760da-4146-4688-a275-418314974b55/657a47b5-711a-4c36-9b6b-73aa4928b137"
-					(reference "#PWR049")
-					(unit 1)
-				)
-				(path "/d5946b96-44a8-4a28-8641-19803e1510af/ab4760da-4146-4688-a275-418314974b55/207d6e2c-5657-4cae-9098-bf31bbf0eeb3/9d425879-c049-4dfa-82be-004c8041dfbb"
-					(reference "#PWR046")
-					(unit 1)
-				)
-				(path "/d5946b96-44a8-4a28-8641-19803e1510af/ab4760da-4146-4688-a275-418314974b55/216077bc-1e97-451f-9a4f-0a4e0691e85e/9d425879-c049-4dfa-82be-004c8041dfbb"
-					(reference "#PWR0111")
+					(reference "#PWR048")
+					(unit 1)
+				)
+				(path "/d5946b96-44a8-4a28-8641-19803e1510af/ab4760da-4146-4688-a275-418314974b55/207d6e2c-5657-4cae-9098-bf31bbf0eeb3/9d425879-c049-4dfa-82be-004c8041dfbb"
+					(reference "#PWR045")
+					(unit 1)
+				)
+				(path "/d5946b96-44a8-4a28-8641-19803e1510af/ab4760da-4146-4688-a275-418314974b55/216077bc-1e97-451f-9a4f-0a4e0691e85e/9d425879-c049-4dfa-82be-004c8041dfbb"
+					(reference "#PWR0109")
 					(unit 1)
 				)
@@
 		(dnp no)
 		(fields_autoplaced yes)
-		(property "Reference" "R22"
+		(property "Reference" "R23"
 			(at 129.54 91.44 90)
 			(effects
@@
 			(project "apple_peeler_pcb"
 				(path "/d5946b96-44a8-4a28-8641-19803e1510af/ab4760da-4146-4688-a275-418314974b55/657a47b5-711a-4c36-9b6b-73aa4928b137"
-					(reference "R25")
-					(unit 1)
-				)
-				(path "/d5946b96-44a8-4a28-8641-19803e1510af/ab4760da-4146-4688-a275-418314974b55/207d6e2c-5657-4cae-9098-bf31bbf0eeb3/9d425879-c049-4dfa-82be-004c8041dfbb"
-					(reference "R22")
-					(unit 1)
-				)
-				(path "/d5946b96-44a8-4a28-8641-19803e1510af/ab4760da-4146-4688-a275-418314974b55/216077bc-1e97-451f-9a4f-0a4e0691e85e/9d425879-c049-4dfa-82be-004c8041dfbb"
-					(reference "R44")
+					(reference "R26")
+					(unit 1)
+				)
+				(path "/d5946b96-44a8-4a28-8641-19803e1510af/ab4760da-4146-4688-a275-418314974b55/207d6e2c-5657-4cae-9098-bf31bbf0eeb3/9d425879-c049-4dfa-82be-004c8041dfbb"
+					(reference "R23")
+					(unit 1)
+				)
+				(path "/d5946b96-44a8-4a28-8641-19803e1510af/ab4760da-4146-4688-a275-418314974b55/216077bc-1e97-451f-9a4f-0a4e0691e85e/9d425879-c049-4dfa-82be-004c8041dfbb"
+					(reference "R45")
 					(unit 1)
 				)
@@
 		(dnp no)
 		(fields_autoplaced yes)
-		(property "Reference" "R24"
+		(property "Reference" "R25"
 			(at 143.51 82.5499 0)
 			(effects
@@
 			(project "apple_peeler_pcb"
 				(path "/d5946b96-44a8-4a28-8641-19803e1510af/ab4760da-4146-4688-a275-418314974b55/657a47b5-711a-4c36-9b6b-73aa4928b137"
-					(reference "R27")
-					(unit 1)
-				)
-				(path "/d5946b96-44a8-4a28-8641-19803e1510af/ab4760da-4146-4688-a275-418314974b55/207d6e2c-5657-4cae-9098-bf31bbf0eeb3/9d425879-c049-4dfa-82be-004c8041dfbb"
-					(reference "R24")
-					(unit 1)
-				)
-				(path "/d5946b96-44a8-4a28-8641-19803e1510af/ab4760da-4146-4688-a275-418314974b55/216077bc-1e97-451f-9a4f-0a4e0691e85e/9d425879-c049-4dfa-82be-004c8041dfbb"
-					(reference "R46")
+					(reference "R28")
+					(unit 1)
+				)
+				(path "/d5946b96-44a8-4a28-8641-19803e1510af/ab4760da-4146-4688-a275-418314974b55/207d6e2c-5657-4cae-9098-bf31bbf0eeb3/9d425879-c049-4dfa-82be-004c8041dfbb"
+					(reference "R25")
+					(unit 1)
+				)
+				(path "/d5946b96-44a8-4a28-8641-19803e1510af/ab4760da-4146-4688-a275-418314974b55/216077bc-1e97-451f-9a4f-0a4e0691e85e/9d425879-c049-4dfa-82be-004c8041dfbb"
+					(reference "R47")
 					(unit 1)
 				)
@@
 		(on_board yes)
 		(dnp no)
-		(property "Reference" "#PWR048"
+		(property "Reference" "#PWR047"
 			(at 146.05 116.84 0)
 			(effects
@@
 			(project "apple_peeler_pcb"
 				(path "/d5946b96-44a8-4a28-8641-19803e1510af/ab4760da-4146-4688-a275-418314974b55/657a47b5-711a-4c36-9b6b-73aa4928b137"
-					(reference "#PWR051")
-					(unit 1)
-				)
-				(path "/d5946b96-44a8-4a28-8641-19803e1510af/ab4760da-4146-4688-a275-418314974b55/207d6e2c-5657-4cae-9098-bf31bbf0eeb3/9d425879-c049-4dfa-82be-004c8041dfbb"
-					(reference "#PWR048")
-					(unit 1)
-				)
-				(path "/d5946b96-44a8-4a28-8641-19803e1510af/ab4760da-4146-4688-a275-418314974b55/216077bc-1e97-451f-9a4f-0a4e0691e85e/9d425879-c049-4dfa-82be-004c8041dfbb"
-					(reference "#PWR0113")
+					(reference "#PWR050")
+					(unit 1)
+				)
+				(path "/d5946b96-44a8-4a28-8641-19803e1510af/ab4760da-4146-4688-a275-418314974b55/207d6e2c-5657-4cae-9098-bf31bbf0eeb3/9d425879-c049-4dfa-82be-004c8041dfbb"
+					(reference "#PWR047")
+					(unit 1)
+				)
+				(path "/d5946b96-44a8-4a28-8641-19803e1510af/ab4760da-4146-4688-a275-418314974b55/216077bc-1e97-451f-9a4f-0a4e0691e85e/9d425879-c049-4dfa-82be-004c8041dfbb"
+					(reference "#PWR0111")
 					(unit 1)
 				)
@@
 		(dnp no)
 		(fields_autoplaced yes)
-		(property "Reference" "R23"
+		(property "Reference" "R24"
 			(at 138.43 104.1399 0)
 			(effects
@@
 			(project "apple_peeler_pcb"
 				(path "/d5946b96-44a8-4a28-8641-19803e1510af/ab4760da-4146-4688-a275-418314974b55/657a47b5-711a-4c36-9b6b-73aa4928b137"
-					(reference "R26")
-					(unit 1)
-				)
-				(path "/d5946b96-44a8-4a28-8641-19803e1510af/ab4760da-4146-4688-a275-418314974b55/207d6e2c-5657-4cae-9098-bf31bbf0eeb3/9d425879-c049-4dfa-82be-004c8041dfbb"
-					(reference "R23")
-					(unit 1)
-				)
-				(path "/d5946b96-44a8-4a28-8641-19803e1510af/ab4760da-4146-4688-a275-418314974b55/216077bc-1e97-451f-9a4f-0a4e0691e85e/9d425879-c049-4dfa-82be-004c8041dfbb"
-					(reference "R45")
+					(reference "R27")
+					(unit 1)
+				)
+				(path "/d5946b96-44a8-4a28-8641-19803e1510af/ab4760da-4146-4688-a275-418314974b55/207d6e2c-5657-4cae-9098-bf31bbf0eeb3/9d425879-c049-4dfa-82be-004c8041dfbb"
+					(reference "R24")
+					(unit 1)
+				)
+				(path "/d5946b96-44a8-4a28-8641-19803e1510af/ab4760da-4146-4688-a275-418314974b55/216077bc-1e97-451f-9a4f-0a4e0691e85e/9d425879-c049-4dfa-82be-004c8041dfbb"
+					(reference "R46")
 					(unit 1)
 				)
@@
 		(on_board yes)
 		(dnp no)
-		(property "Reference" "#PWR047"
+		(property "Reference" "#PWR046"
 			(at 146.05 82.55 0)
 			(effects
@@
 			(project "apple_peeler_pcb"
 				(path "/d5946b96-44a8-4a28-8641-19803e1510af/ab4760da-4146-4688-a275-418314974b55/657a47b5-711a-4c36-9b6b-73aa4928b137"
-					(reference "#PWR050")
-					(unit 1)
-				)
-				(path "/d5946b96-44a8-4a28-8641-19803e1510af/ab4760da-4146-4688-a275-418314974b55/207d6e2c-5657-4cae-9098-bf31bbf0eeb3/9d425879-c049-4dfa-82be-004c8041dfbb"
-					(reference "#PWR047")
-					(unit 1)
-				)
-				(path "/d5946b96-44a8-4a28-8641-19803e1510af/ab4760da-4146-4688-a275-418314974b55/216077bc-1e97-451f-9a4f-0a4e0691e85e/9d425879-c049-4dfa-82be-004c8041dfbb"
-					(reference "#PWR0112")
-					(unit 1)
-				)
+					(reference "#PWR049")
+					(unit 1)
+				)
+				(path "/d5946b96-44a8-4a28-8641-19803e1510af/ab4760da-4146-4688-a275-418314974b55/207d6e2c-5657-4cae-9098-bf31bbf0eeb3/9d425879-c049-4dfa-82be-004c8041dfbb"
+					(reference "#PWR046")
+					(unit 1)
+				)
+				(path "/d5946b96-44a8-4a28-8641-19803e1510af/ab4760da-4146-4688-a275-418314974b55/216077bc-1e97-451f-9a4f-0a4e0691e85e/9d425879-c049-4dfa-82be-004c8041dfbb"
+					(reference "#PWR0110")
+					(unit 1)
+				)
