File: apple_peeler_pcb/usb.kicad_sch (KiCad schematic)
At the start: 5 parts, among them J5 USB_C_Receptacle_USB2.0_16P

Commit message: use wleds instead of individual leds
Parts:
- renumbered R43 to R38, R44 to R39, R45 to R40, R46 to R41
Changed lines of the file:
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@@
 		(dnp no)
 		(fields_autoplaced yes)
-		(property "Reference" "#PWR070"
+		(property "Reference" "#PWR065"
 			(at 143.51 132.08 0)
 			(effects
@@
 			(project "apple_peeler_pcb"
 				(path "/d5946b96-44a8-4a28-8641-19803e1510af/755a6c0d-ab83-4668-9075-6ff3f25fd8c2"
-					(reference "#PWR070")
+					(reference "#PWR065")
 					(unit 1)
 				)
@@
 		(on_board yes)
 		(dnp no)
-		(property "Reference" "R45"
+		(property "Reference" "R40"
 			(at 173.99 92.71 90)
 			(effects
@@
 			(project "apple_peeler_pcb"
 				(path "/d5946b96-44a8-4a28-8641-19803e1510af/755a6c0d-ab83-4668-9075-6ff3f25fd8c2"
-					(reference "R45")
+					(reference "R40")
 					(unit 1)
 				)
@@
 		(on_board yes)
 		(dnp no)
-		(property "Reference" "R46"
+		(property "Reference" "R41"
 			(at 173.99 97.79 90)
 			(effects
@@
 			(project "apple_peeler_pcb"
 				(path "/d5946b96-44a8-4a28-8641-19803e1510af/755a6c0d-ab83-4668-9075-6ff3f25fd8c2"
-					(reference "R46")
+					(reference "R41")
 					(unit 1)
 				)
@@
 		(dnp no)
 		(fields_autoplaced yes)
-		(property "Reference" "R44"
+		(property "Reference" "R39"
 			(at 157.48 111.7599 0)
 			(effects
@@
 			(project "apple_peeler_pcb"
 				(path "/d5946b96-44a8-4a28-8641-19803e1510af/755a6c0d-ab83-4668-9075-6ff3f25fd8c2"
-					(reference "R44")
+					(reference "R39")
 					(unit 1)
 				)
@@
 		(dnp no)
 		(fields_autoplaced yes)
-		(property "Reference" "#PWR069"
+		(property "Reference" "#PWR064"
 			(at 123.19 132.08 0)
 			(effects
@@
 			(project "apple_peeler_pcb"
 				(path "/d5946b96-44a8-4a28-8641-19803e1510af/755a6c0d-ab83-4668-9075-6ff3f25fd8c2"
-					(reference "#PWR069")
+					(reference "#PWR064")
 					(unit 1)
 				)
@@
 		(dnp no)
 		(fields_autoplaced yes)
-		(property "Reference" "R43"
+		(property "Reference" "R38"
 			(at 146.05 111.7599 0)
 			(effects
@@
 			(project "apple_peeler_pcb"
 				(path "/d5946b96-44a8-4a28-8641-19803e1510af/755a6c0d-ab83-4668-9075-6ff3f25fd8c2"
-					(reference "R43")
+					(reference "R38")
 					(unit 1)
 				)
@@
 		(dnp no)
 		(fields_autoplaced yes)
-		(property "Reference" "#PWR068"
+		(property "Reference" "#PWR063"
 			(at 115.57 132.08 0)
 			(effects
@@
 			(project "apple_peeler_pcb"
 				(path "/d5946b96-44a8-4a28-8641-19803e1510af/755a6c0d-ab83-4668-9075-6ff3f25fd8c2"
-					(reference "#PWR068")
+					(reference "#PWR063")
 					(unit 1)
 				)
@@
 		(dnp no)
 		(fields_autoplaced yes)
-		(property "Reference" "#PWR071"
+		(property "Reference" "#PWR066"
 			(at 154.94 132.08 0)
 			(effects
@@
 			(project "apple_peeler_pcb"
 				(path "/d5946b96-44a8-4a28-8641-19803e1510af/755a6c0d-ab83-4668-9075-6ff3f25fd8c2"
-					(reference "#PWR071")
-					(unit 1)
-				)
+					(reference "#PWR066")
+					(unit 1)
+				)

Commit message: some progress
Connections:
- net DM renamed DN
Changed lines of the file:
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@@
 		)
 	)
-	(hierarchical_label "DM"
+	(hierarchical_label "DN"
 		(shape bidirectional)
 		(at 184.15 100.33 0)

Commit message: add loads of test points
Parts:
- renumbered J5 to J7
Changed lines of the file:
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@@
 		(dnp no)
 		(fields_autoplaced yes)
-		(property "Reference" "#PWR065"
+		(property "Reference" "#PWR067"
 			(at 143.51 132.08 0)
 			(effects
@@
 			(project "apple_peeler_pcb"
 				(path "/d5946b96-44a8-4a28-8641-19803e1510af/755a6c0d-ab83-4668-9075-6ff3f25fd8c2"
-					(reference "#PWR065")
+					(reference "#PWR067")
 					(unit 1)
 				)
@@
 		(dnp no)
 		(fields_autoplaced yes)
-		(property "Reference" "#PWR064"
+		(property "Reference" "#PWR066"
 			(at 123.19 132.08 0)
 			(effects
@@
 			(project "apple_peeler_pcb"
 				(path "/d5946b96-44a8-4a28-8641-19803e1510af/755a6c0d-ab83-4668-9075-6ff3f25fd8c2"
-					(reference "#PWR064")
+					(reference "#PWR066")
 					(unit 1)
 				)
@@
 		(dnp no)
 		(fields_autoplaced yes)
-		(property "Reference" "#PWR063"
+		(property "Reference" "#PWR065"
 			(at 115.57 132.08 0)
 			(effects
@@
 			(project "apple_peeler_pcb"
 				(path "/d5946b96-44a8-4a28-8641-19803e1510af/755a6c0d-ab83-4668-9075-6ff3f25fd8c2"
-					(reference "#PWR063")
+					(reference "#PWR065")
 					(unit 1)
 				)
@@
 		(dnp no)
 		(fields_autoplaced yes)
-		(property "Reference" "J5"
+		(property "Reference" "J7"
 			(at 123.19 74.93 0)
 			(effects
@@
 			(project ""
 				(path "/d5946b96-44a8-4a28-8641-19803e1510af/755a6c0d-ab83-4668-9075-6ff3f25fd8c2"
-					(reference "J5")
+					(reference "J7")
 					(unit 1)
 				)
@@
 		(dnp no)
 		(fields_autoplaced yes)
-		(property "Reference" "#PWR066"
+		(property "Reference" "#PWR068"
 			(at 154.94 132.08 0)
 			(effects
@@
 			(project "apple_peeler_pcb"
 				(path "/d5946b96-44a8-4a28-8641-19803e1510af/755a6c0d-ab83-4668-9075-6ff3f25fd8c2"
-					(reference "#PWR066")
-					(unit 1)
-				)
+					(reference "#PWR068")
+					(unit 1)
+				)

Commit message: reroute SMPS layout by closely following datasheet
Connections:
- net USB_SIDE_DP: now reaches J7.A7 (D-), J7.B7 (D-), R40.1
- net USB_SIDE_DN: now reaches J7.A6 (D+), J7.B6 (D+), R41.1
Other:
- moved on the sheet: R40, R41
Changed lines of the file:
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@@
 	(wire
 		(pts
-			(xy 177.8 95.25) (xy 184.15 95.25)
+			(xy 201.93 95.25) (xy 208.28 95.25)
 		)
 		(stroke
@@
 	(wire
 		(pts
-			(xy 177.8 100.33) (xy 184.15 100.33)
+			(xy 201.93 100.33) (xy 208.28 100.33)
 		)
 		(stroke
@@
 	(wire
 		(pts
-			(xy 140.97 95.25) (xy 170.18 95.25)
+			(xy 140.97 95.25) (xy 194.31 95.25)
 		)
 		(stroke
@@
 	(wire
 		(pts
-			(xy 140.97 100.33) (xy 170.18 100.33)
-		)
-		(stroke
-			(width 0)
-			(type default)
+			(xy 140.97 100.33) (xy 194.31 100.33)
+		)
+		(stroke
+			(width 0)
+			(type default)
+		)
+	)
+	(label "USB_SIDE_DN"
+		(at 171.45 100.33 0)
+		(effects
+			(font
+				(size 1.27 1.27)
+			)
+			(justify left bottom)
+		)
+	)
+	(label "USB_SIDE_DP"
+		(at 171.45 95.25 0)
+		(effects
+			(font
+				(size 1.27 1.27)
+			)
+			(justify left bottom)
 		)
 	)
@@
 	(hierarchical_label "DN"
 		(shape bidirectional)
-		(at 184.15 100.33 0)
+		(at 208.28 100.33 0)
 		(effects
 			(font
@@
 	(hierarchical_label "DP"
 		(shape bidirectional)
-		(at 184.15 95.25 0)
+		(at 208.28 95.25 0)
 		(effects
 			(font
@@
 		(polyline
 			(pts
-				(xy 181.61 104.14) (xy 181.61 90.17) (xy 166.37 90.17) (xy 166.37 104.14)
+				(xy 205.74 104.14) (xy 205.74 90.17) (xy 190.5 90.17) (xy 190.5 104.14)
 			)
 			(stroke
@@
 		(length 2.54)
 		(shape round)
-		(at 173.99 90.17 0)
+		(at 198.12 90.17 0)
 		(effects
 			(font
@@
 		)
 		(property "Netclass" "USB"
-			(at 172.466 87.63 0)
+			(at 196.596 87.63 0)
 			(effects
 				(font
@@
 		)
 		(property "Component Class" ""
-			(at 476.25 208.28 0)
+			(at 500.38 208.28 0)
 			(effects
 				(font
@@
 	(symbol
 		(lib_id "Device:R")
-		(at 173.99 95.25 90)
+		(at 198.12 95.25 90)
 		(unit 1)
 		(exclude_from_sim no)
@@
 		(dnp no)
 		(property "Reference" "R40"
-			(at 173.99 92.71 90)
+			(at 198.12 92.71 90)
 			(effects
 				(font
@@
 		)
 		(property "Value" "27Ω"
-			(at 173.99 95.25 90)
+			(at 198.12 95.25 90)
 			(effects
 				(font
@@
 		)
 		(property "Footprint" "Resistor_SMD:R_0805_2012Metric"
-			(at 173.99 97.028 90)
+			(at 198.12 97.028 90)
 			(effects
 				(font
@@
 		)
 		(property "Datasheet" "~"
-			(at 173.99 95.25 0)
+			(at 198.12 95.25 0)
 			(effects
 				(font
@@
 		)
 		(property "Description" "Resistor"
-			(at 173.99 95.25 0)
+			(at 198.12 95.25 0)
 			(effects
 				(font
@@
 		)
 		(property "MPN" "R 27Ω 125mW 0805"
-			(at 173.99 95.25 0)
+			(at 198.12 95.25 0)
 			(effects
 				(font
@@
 		)
 		(property "LCSC" "C17594"
-			(at 173.99 95.25 0)
+			(at 198.12 95.25 0)
 			(effects
 				(font
@@
 	(symbol
 		(lib_id "Device:R")
-		(at 173.99 100.33 90)
+		(at 198.12 100.33 90)
 		(unit 1)
 		(exclude_from_sim no)
@@
 		(dnp no)
 		(property "Reference" "R41"
-			(at 173.99 97.79 90)
+			(at 198.12 97.79 90)
 			(effects
 				(font
@@
 		)
 		(property "Value" "27Ω"
-			(at 173.99 100.33 90)
+			(at 198.12 100.33 90)
 			(effects
 				(font
@@
 		)
 		(property "Footprint" "Resistor_SMD:R_0805_2012Metric"
-			(at 173.99 102.108 90)
+			(at 198.12 102.108 90)
 			(effects
 				(font
@@
 		)
 		(property "Datasheet" "~"
-			(at 173.99 100.33 0)
+			(at 198.12 100.33 0)
 			(effects
 				(font
@@
 		)
 		(property "Description" "Resistor"
-			(at 173.99 100.33 0)
+			(at 198.12 100.33 0)
 			(effects
 				(font
@@
 		)
 		(property "MPN" "R 27Ω 125mW 0805"
-			(at 173.99 100.33 0)
+			(at 198.12 100.33 0)
 			(effects
 				(font
@@
 		)
 		(property "LCSC" "C17594"
-			(at 173.99 100.33 0)
-			(effects
-				(font
+			(at 198.12 100.33 0)
+			(effects
+				(font

Commit message: fix connector labels and misc silkscreen
Parts:
- renumbered J7 to J8
Changed lines of the file:
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@@
 		(dnp no)
 		(fields_autoplaced yes)
-		(property "Reference" "#PWR068"
+		(property "Reference" "#PWR069"
 			(at 143.51 132.08 0)
 			(effects
@@
 			(project "apple_peeler_pcb"
 				(path "/d5946b96-44a8-4a28-8641-19803e1510af/755a6c0d-ab83-4668-9075-6ff3f25fd8c2"
-					(reference "#PWR068")
+					(reference "#PWR069")
 					(unit 1)
 				)
@@
 		(dnp no)
 		(fields_autoplaced yes)
-		(property "Reference" "#PWR067"
+		(property "Reference" "#PWR068"
 			(at 123.19 132.08 0)
 			(effects
@@
 			(project "apple_peeler_pcb"
 				(path "/d5946b96-44a8-4a28-8641-19803e1510af/755a6c0d-ab83-4668-9075-6ff3f25fd8c2"
-					(reference "#PWR067")
+					(reference "#PWR068")
 					(unit 1)
 				)
@@
 		(dnp no)
 		(fields_autoplaced yes)
-		(property "Reference" "#PWR066"
+		(property "Reference" "#PWR067"
 			(at 115.57 132.08 0)
 			(effects
@@
 			(project "apple_peeler_pcb"
 				(path "/d5946b96-44a8-4a28-8641-19803e1510af/755a6c0d-ab83-4668-9075-6ff3f25fd8c2"
-					(reference "#PWR066")
+					(reference "#PWR067")
 					(unit 1)
 				)
@@
 		(dnp no)
 		(fields_autoplaced yes)
-		(property "Reference" "J7"
+		(property "Reference" "J8"
 			(at 123.19 74.93 0)
 			(effects
@@
 			(project ""
 				(path "/d5946b96-44a8-4a28-8641-19803e1510af/755a6c0d-ab83-4668-9075-6ff3f25fd8c2"
-					(reference "J7")
+					(reference "J8")
 					(unit 1)
 				)
@@
 		(dnp no)
 		(fields_autoplaced yes)
-		(property "Reference" "#PWR069"
+		(property "Reference" "#PWR070"
 			(at 154.94 132.08 0)
 			(effects
@@
 			(project "apple_peeler_pcb"
 				(path "/d5946b96-44a8-4a28-8641-19803e1510af/755a6c0d-ab83-4668-9075-6ff3f25fd8c2"
-					(reference "#PWR069")
-					(unit 1)
-				)
+					(reference "#PWR070")
+					(unit 1)
+				)

Commit message: replace fancy debug connectors by pin header to save $8
Parts:
- renumbered J8 to J6, R38 to R39, R39 to R40, R40 to R41, R41 to R42
Changed lines of the file:
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@@
 		(dnp no)
 		(fields_autoplaced yes)
-		(property "Reference" "#PWR069"
+		(property "Reference" "#PWR067"
 			(at 143.51 132.08 0)
 			(effects
@@
 			(project "apple_peeler_pcb"
 				(path "/d5946b96-44a8-4a28-8641-19803e1510af/755a6c0d-ab83-4668-9075-6ff3f25fd8c2"
-					(reference "#PWR069")
+					(reference "#PWR067")
 					(unit 1)
 				)
@@
 		(on_board yes)
 		(dnp no)
-		(property "Reference" "R40"
+		(property "Reference" "R41"
 			(at 198.12 92.71 90)
 			(effects
@@
 			(project "apple_peeler_pcb"
 				(path "/d5946b96-44a8-4a28-8641-19803e1510af/755a6c0d-ab83-4668-9075-6ff3f25fd8c2"
-					(reference "R40")
+					(reference "R41")
 					(unit 1)
 				)
@@
 		(on_board yes)
 		(dnp no)
-		(property "Reference" "R41"
+		(property "Reference" "R42"
 			(at 198.12 97.79 90)
 			(effects
@@
 			(project "apple_peeler_pcb"
 				(path "/d5946b96-44a8-4a28-8641-19803e1510af/755a6c0d-ab83-4668-9075-6ff3f25fd8c2"
-					(reference "R41")
+					(reference "R42")
 					(unit 1)
 				)
@@
 		(dnp no)
 		(fields_autoplaced yes)
-		(property "Reference" "R39"
+		(property "Reference" "R40"
 			(at 157.48 111.7599 0)
 			(effects
@@
 			(project "apple_peeler_pcb"
 				(path "/d5946b96-44a8-4a28-8641-19803e1510af/755a6c0d-ab83-4668-9075-6ff3f25fd8c2"
-					(reference "R39")
+					(reference "R40")
 					(unit 1)
 				)
@@
 		(dnp no)
 		(fields_autoplaced yes)
-		(property "Reference" "#PWR068"
+		(property "Reference" "#PWR066"
 			(at 123.19 132.08 0)
 			(effects
@@
 			(project "apple_peeler_pcb"
 				(path "/d5946b96-44a8-4a28-8641-19803e1510af/755a6c0d-ab83-4668-9075-6ff3f25fd8c2"
-					(reference "#PWR068")
+					(reference "#PWR066")
 					(unit 1)
 				)
@@
 		(dnp no)
 		(fields_autoplaced yes)
-		(property "Reference" "R38"
+		(property "Reference" "R39"
 			(at 146.05 111.7599 0)
 			(effects
@@
 			(project "apple_peeler_pcb"
 				(path "/d5946b96-44a8-4a28-8641-19803e1510af/755a6c0d-ab83-4668-9075-6ff3f25fd8c2"
-					(reference "R38")
+					(reference "R39")
 					(unit 1)
 				)
@@
 		(dnp no)
 		(fields_autoplaced yes)
-		(property "Reference" "#PWR067"
+		(property "Reference" "#PWR065"
 			(at 115.57 132.08 0)
 			(effects
@@
 			(project "apple_peeler_pcb"
 				(path "/d5946b96-44a8-4a28-8641-19803e1510af/755a6c0d-ab83-4668-9075-6ff3f25fd8c2"
-					(reference "#PWR067")
+					(reference "#PWR065")
 					(unit 1)
 				)
@@
 		(dnp no)
 		(fields_autoplaced yes)
-		(property "Reference" "J8"
+		(property "Reference" "J6"
 			(at 123.19 74.93 0)
 			(effects
@@
 			(project ""
 				(path "/d5946b96-44a8-4a28-8641-19803e1510af/755a6c0d-ab83-4668-9075-6ff3f25fd8c2"
-					(reference "J8")
+					(reference "J6")
 					(unit 1)
 				)
@@
 		(dnp no)
 		(fields_autoplaced yes)
-		(property "Reference" "#PWR070"
+		(property "Reference" "#PWR068"
 			(at 154.94 132.08 0)
 			(effects
@@
 			(project "apple_peeler_pcb"
 				(path "/d5946b96-44a8-4a28-8641-19803e1510af/755a6c0d-ab83-4668-9075-6ff3f25fd8c2"
-					(reference "#PWR070")
-					(unit 1)
-				)
+					(reference "#PWR068")
+					(unit 1)
+				)

Commit message: fix the fucking fucked D+ and D- lines
Connections:
- net USB_SIDE_DN: now also J6.A7 (D-), J6.B7 (D-); no longer J6.A6 (D+), J6.B6 (D+)
- net USB_SIDE_DP: now also J6.A6 (D+), J6.B6 (D+); no longer J6.A7 (D-), J6.B7 (D-)
Other:
- moved on the sheet: R41, R42
Changed lines of the file:
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@@
 	)
 	(label "USB_SIDE_DN"
-		(at 171.45 100.33 0)
+		(at 170.18 95.25 0)
 		(effects
 			(font
@@
 	)
 	(label "USB_SIDE_DP"
-		(at 171.45 95.25 0)
+		(at 170.18 100.33 0)
 		(effects
 			(font
@@
 	(hierarchical_label "DN"
 		(shape bidirectional)
-		(at 208.28 100.33 0)
+		(at 208.28 95.25 0)
 		(effects
 			(font
@@
 	(hierarchical_label "DP"
 		(shape bidirectional)
-		(at 208.28 95.25 0)
+		(at 208.28 100.33 0)
 		(effects
 			(font
@@
 	(symbol
 		(lib_id "Device:R")
+		(at 198.12 100.33 90)
+		(unit 1)
+		(exclude_from_sim no)
+		(in_bom yes)
+		(on_board yes)
+		(dnp no)
+		(property "Reference" "R41"
+			(at 198.12 97.79 90)
+			(effects
+				(font
+					(size 1.27 1.27)
+				)
+			)
+		)
+		(property "Value" "27Ω"
+			(at 198.12 100.33 90)
+			(effects
+				(font
+					(size 1.27 1.27)
+				)
+			)
+		)
+		(property "Footprint" "Resistor_SMD:R_0805_2012Metric"
+			(at 198.12 102.108 90)
+			(effects
+				(font
+					(size 1.27 1.27)
+				)
+				(hide yes)
+			)
+		)
+		(property "Datasheet" "~"
+			(at 198.12 100.33 0)
+			(effects
+				(font
+					(size 1.27 1.27)
+				)
+				(hide yes)
+			)
+		)
+		(property "Description" "Resistor"
+			(at 198.12 100.33 0)
+			(effects
+				(font
+					(size 1.27 1.27)
+				)
+				(hide yes)
+			)
+		)
+		(property "MPN" "R 27Ω 125mW 0805"
+			(at 198.12 100.33 0)
+			(effects
+				(font
+					(size 1.27 1.27)
+				)
+				(hide yes)
+			)
+		)
+		(property "LCSC" "C17594"
+			(at 198.12 100.33 0)
+			(effects
+				(font
+					(size 1.27 1.27)
+				)
+				(hide yes)
+			)
+		)
+		(pin "1"
+		)
+		(pin "2"
+		)
+		(instances
+			(project "apple_peeler_pcb"
+				(path "/d5946b96-44a8-4a28-8641-19803e1510af/755a6c0d-ab83-4668-9075-6ff3f25fd8c2"
+					(reference "R41")
+					(unit 1)
+				)
+			)
+		)
+	)
+	(symbol
+		(lib_id "Device:R")
 		(at 198.12 95.25 90)
 		(unit 1)
@@
 		(on_board yes)
 		(dnp no)
-		(property "Reference" "R41"
+		(property "Reference" "R42"
 			(at 198.12 92.71 90)
 			(effects
@@
 			(effects
 				(font
-					(size 1.27 1.27)
-				)
-				(hide yes)
-			)
-		)
-		(pin "1"
-		)
-		(pin "2"
-		)
-		(instances
-			(project "apple_peeler_pcb"
-				(path "/d5946b96-44a8-4a28-8641-19803e1510af/755a6c0d-ab83-4668-9075-6ff3f25fd8c2"
-					(reference "R41")
-					(unit 1)
-				)
-			)
-		)
-	)
-	(symbol
-		(lib_id "Device:R")
-		(at 198.12 100.33 90)
-		(unit 1)
-		(exclude_from_sim no)
-		(in_bom yes)
-		(on_board yes)
-		(dnp no)
-		(property "Reference" "R42"
-			(at 198.12 97.79 90)
-			(effects
-				(font
-					(size 1.27 1.27)
-				)
-			)
-		)
-		(property "Value" "27Ω"
-			(at 198.12 100.33 90)
-			(effects
-				(font
-					(size 1.27 1.27)
-				)
-			)
-		)
-		(property "Footprint" "Resistor_SMD:R_0805_2012Metric"
-			(at 198.12 102.108 90)
-			(effects
-				(font
-					(size 1.27 1.27)
-				)
-				(hide yes)
-			)
-		)
-		(property "Datasheet" "~"
-			(at 198.12 100.33 0)
-			(effects
-				(font
-					(size 1.27 1.27)
-				)
-				(hide yes)
-			)
-		)
-		(property "Description" "Resistor"
-			(at 198.12 100.33 0)
-			(effects
-				(font
-					(size 1.27 1.27)
-				)
-				(hide yes)
-			)
-		)
-		(property "MPN" "R 27Ω 125mW 0805"
-			(at 198.12 100.33 0)
-			(effects
-				(font
-					(size 1.27 1.27)
-				)
-				(hide yes)
-			)
-		)
-		(property "LCSC" "C17594"
-			(at 198.12 100.33 0)
-			(effects
-				(font
