File: apple_peeler_pcb/usb.kicad_sch (KiCad schematic)
At the start: 5 parts, among them J6 USB_C_Receptacle_USB2.0_16P

Commit message: fix the fucking WLED footprints
Parts:
- renumbered R42 to R41, R41 to R42
Changed lines of the file:
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@@
 		(on_board yes)
 		(dnp no)
-		(property "Reference" "R41"
+		(property "Reference" "R42"
 			(at 198.12 97.79 90)
 			(effects
@@
 			(project "apple_peeler_pcb"
 				(path "/d5946b96-44a8-4a28-8641-19803e1510af/755a6c0d-ab83-4668-9075-6ff3f25fd8c2"
-					(reference "R41")
+					(reference "R42")
 					(unit 1)
 				)
@@
 		(on_board yes)
 		(dnp no)
-		(property "Reference" "R42"
+		(property "Reference" "R41"
 			(at 198.12 92.71 90)
 			(effects
@@
 			(project "apple_peeler_pcb"
 				(path "/d5946b96-44a8-4a28-8641-19803e1510af/755a6c0d-ab83-4668-9075-6ff3f25fd8c2"
-					(reference "R42")
+					(reference "R41")
 					(unit 1)
 				)
